File: adapter/adapter.kicad_pcb (KiCad board)
At the start: 2 copper layers, 93.5 x 50.9 mm, 64 parts, among them J1 Serial, J10 Ribbon, J11 Ribbon, J12 Ribbon, J13 serial, J14 serial, J2 Serial, J3 battery charge, J4 RGB, J5 RGB, J6 battery charge, J7 trackball, J8 trackball, J9 Ribbon, SW1 SW_SPST, SW2 SW_SPST, SW3 SW_SPDT, SW4 SW_SPDT, U1 eliteC, U2 eliteC

Commit message: RP2040 mods made
Parts:
- removed G*** (x2): LOGO, LOGO
- removed J13, J14: serial, Library:PinHeader_1x04_P2.54mm_Vertical
- removed J3, J6: battery charge, Library:PinHeader_1x02_P2.54mm_Vertical
- removed J7, J8: trackball, Library:6_PinHeader
- removed JP1, JP2: Jumper_2_Open, Library:power_switch_jumper
- removed R1, R3, R5, R6: 5.1k, Library:R_1206_handsolder
- removed R2, R4: 4.7k, Library:R_1206_handsolder
- removed SW3, SW4: SW_SPDT, Library:SW_SPDT+H-MSK12C01_hor(7pin_SMD)
- removed U1, U2: eliteC, Library:Elite-C
- removed the kibuzzard-61F01957 at (189.4, 100.3)
- removed the kibuzzard-61F01957 at (121.2, 100.3)
- removed kibuzzard-61F01C84 (x2): G***, kibuzzard-61F01C84
- removed kibuzzard-6208EDFE: G***, kibuzzard-6208EDFE
- removed kibuzzard-6208EE22: G***, kibuzzard-6208EE22
- removed kibuzzard-62093EDE: G***, kibuzzard-62093EDE
- removed kibuzzard-62094D1C: G***, kibuzzard-62094D1C
- removed kibuzzard-620B8593 (x2): G***, kibuzzard-620B8593
- removed kibuzzard-620B8D91 (x4): G***, kibuzzard-620B8D91
- added RZ1: RP2040-Zero, KB Parts:RP2040-Zero, F.Cu at (124.2, 91.8)
- added RZ2: RP2040-Zero, KB Parts:RP2040-Zero, F.Cu at (168.9, 91.8)
- SW1, SW2: value SW_SPST -> SW_Push; footprint Library:PushSwitch -> Keebio Parts:SW_Tactile_SPST_Angled_MJTP1117
- moved SW2 14.1 mm to (180.4, 75.5), turned to 180 degrees
- moved SW1 12.9 mm to (135.3, 76.6), turned to 180 degrees
- moved J10 6.47 mm to (126.2, 102.6)
- moved J9 4.97 mm to (132.8, 102.7)
- moved kibuzzard-6208EFFE 0.71 mm to (177.4, 70.5)
- moved kibuzzard-6208EFFE 0.71 mm to (177.4, 70.3)
- moved kibuzzard-61F01B61 0.26 mm to (132.9, 70.2)
- moved kibuzzard-61F01B61 0.26 mm to (132.7, 70.2)
Connections:
- J1 pad R1: GND -> sda_l
- J1 pad R2: serial_l -> scl_l
- J1 pad S: unconnected-(J1-PadS) -> GND
- J10 pad 1: row4_l -> row1_l
- J10 pad 2: row3_l -> col2_l
- J10 pad 3: col4_l -> col1_l
- J10 pad 4: col5_l -> row2_l
- J10 pad 5: col6_l -> col3_l
- J11 pad 1: col3_r -> row4_r
- J11 pad 2: row1_r -> row3_r
- J11 pad 3: col2_r -> col4_r
- J11 pad 4: col1_r -> col5_r
- J11 pad 5: row2_r -> col6_r
- J12 pad 1: row4_r -> row1_r
- J12 pad 2: row3_r -> col2_r
- J12 pad 3: col4_r -> col1_r
- J12 pad 4: col5_r -> row2_r
- J12 pad 5: col6_r -> col3_r
- J2 pad R1: GND -> scl_r
- J2 pad R2: serial_r -> sda_r
- J2 pad S: unconnected-(J2-PadS) -> GND
- J9 pad 1: col3_l -> row4_l
- J9 pad 2: row1_l -> row3_l
- J9 pad 3: col2_l -> col4_l
- J9 pad 4: col1_l -> col5_l
- J9 pad 5: row2_l -> col6_l
- SW1 pad 1: Rst -> rst_l
- SW2 pad 1: Rst2 -> rst_r
Routing:
- net GND: track 0.00 -> 67.3 mm, vias 0 -> 2
- net miso_r: track 54.1 -> 0.00 mm, vias 1 -> 0
- net mosi_r: track 49.5 -> 0.00 mm, vias 1 -> 0
- net ss_r: track 49.0 -> 0.00 mm, vias 1 -> 0
- net sc_r: track 48.4 -> 0.00 mm, vias 1 -> 0
- net +5V: track 108.3 -> 76.3 mm
- net Rst2: track 30.0 -> 0.00 mm, vias 2 -> 0
- net split_hand_r: track 28.5 -> 0.00 mm, vias 1 -> 0
- net split_hand_l: track 26.5 -> 0.00 mm, vias 2 -> 0
- net miso_l: track 24.0 -> 0.00 mm
- net sc_l: track 23.7 -> 0.00 mm
- net serial_l: track 22.1 -> 0.00 mm
- net Rst: track 20.3 -> 0.00 mm
- net mosi_l: track 18.1 -> 0.00 mm
- net bat_sw_l: track 16.2 -> 0.00 mm, vias 1 -> 0
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Other:
- outline, holes or cut-outs redrawn
- board text added: "Install RP2040-Zero and trs jack face up on this side. Reset button on the opposite."
- board text added: "RP2040 Zero HOLDER 2.1"
- board text added: "mods by mohoyt"
- board text removed: "4.7k"
- board text removed: "B+"
- board text removed: "B-"
- board text removed: "CS"
- board text removed: "ELITE-C HOLDER 2.1"
- board text removed: "Install Elite-C upside down together with ribbon cables and trs jack on this side. Push button on the opposite."
- board text removed: "MISO"
- board text removed: "MOSI"
- board text removed: "S"
- board text removed: "SCL"
- board text removed: "SCLK"
- board text removed: "SDA"
- board text removed: "Special thanks to: Drashna, Freznel Karl"
