File: adapter/adapter.kicad_sch (KiCad schematic)
At the start: 32 parts, among them J1 Serial, J10 Ribbon, J11 Ribbon, J12 Ribbon, J13 serial, J14 serial, J2 Serial, J3 battery charge, J4 RGB, J5 RGB, J6 battery charge, J7 trackball, J8 trackball, J9 Ribbon, SW1 SW_SPST, SW2 SW_SPST, SW3 SW_SPDT, SW4 SW_SPDT, U1 eliteC, U2 eliteC

Commit message: RP2040 mods made
Parts:
- removed J13, J14: serial, Library:PinHeader_1x04_P2.54mm_Vertical, symbol Connector:Conn_01x04_Female
- removed J3, J6: battery charge, Library:PinHeader_1x02_P2.54mm_Vertical, symbol Connector:Conn_01x02_Female
- removed J7, J8: trackball, Library:6_PinHeader, symbol Connector:Conn_01x06_Female
- removed JP1, JP2: Jumper_2_Open, Library:power_switch_jumper, symbol Jumper:Jumper_2_Open
- removed R1, R3, R5, R6: 5.1k, Library:R_1206_handsolder, symbol Device:R
- removed R2, R4: 4.7k, Library:R_1206_handsolder, symbol Device:R
- removed SW1, SW2: SW_SPST, Library:PushSwitch, symbol Switch:SW_SPST
- removed SW3, SW4: SW_SPDT, Library:SW_SPDT+H-MSK12C01_hor(7pin_SMD), symbol Switch:SW_SPDT
- removed U1, U2: eliteC, Library:Elite-C, symbol elite-C:eliteC
- added RZ1, RZ2: RP2040-Zero, KB Parts:RP2040-Zero, symbol rp2040-zero:RP2040-Zero
- added SW1, SW2: SW_Push, Keebio Parts:SW_SPST_3x3, symbol Switch:SW_Push
Connections:
- net serial_l is gone; now on net scl_l: J1.R2
- net serial_r is gone; now on net sda_r: J2.R2
- net +5V: now also RZ1.22 (5V), RZ2.22 (5V)
- net GND: now also J1.S, J2.S, RZ1.23 (GND), RZ2.23 (GND), SW1.2, SW2.2; no longer J1.R1, J2.R1
- net col1_l: now also J10.3 (Pin_3), RZ1.18 (GP27); no longer J9.4 (Pin_4)
- net col1_r: now also J12.3 (Pin_3), RZ2.18 (GP27); no longer J11.4 (Pin_4)
- net col2_l: now also J10.2 (Pin_2), RZ1.19 (GP28); no longer J9.3 (Pin_3)
- net col2_r: now also J12.2 (Pin_2), RZ2.19 (GP28); no longer J11.3 (Pin_3)
- net col3_l: now also J10.5 (Pin_5), RZ1.16 (GP15); no longer J9.1 (Pin_1)
- net col3_r: now also J12.5 (Pin_5), RZ2.16 (GP15); no longer J11.1 (Pin_1)
- net col4_l: now also J9.3 (Pin_3), RZ1.7 (GP6); no longer J10.3 (Pin_3)
- net col4_r: now also J11.3 (Pin_3), RZ2.7 (GP6); no longer J12.3 (Pin_3)
- net col5_l: now also J9.4 (Pin_4), RZ1.8 (GP7); no longer J10.4 (Pin_4)
- net col5_r: now also J11.4 (Pin_4), RZ2.8 (GP7); no longer J12.4 (Pin_4)
- net col6_l: now also J9.5 (Pin_5), RZ1.9 (GP8); no longer J10.5 (Pin_5)
- net col6_r: now also J11.5 (Pin_5), RZ2.9 (GP8); no longer J12.5 (Pin_5)
- net rgb_l: now also RZ2.1 (GP0)
- net rgb_r: now also RZ1.1 (GP0)
- net row1_l: now also J10.1 (Pin_1), RZ1.20 (GP29); no longer J9.2 (Pin_2)
- net row1_r: now also J12.1 (Pin_1), RZ2.20 (GP29); no longer J11.2 (Pin_2)
- net row2_l: now also J10.4 (Pin_4), RZ1.17 (GP26); no longer J9.5 (Pin_5)
- net row2_r: now also J12.4 (Pin_4), RZ2.17 (GP26); no longer J11.5 (Pin_5)
- net row3_l: now also J9.2 (Pin_2), RZ1.6 (GP5); no longer J10.2 (Pin_2)
- net row3_r: now also J11.2 (Pin_2), RZ2.6 (GP5); no longer J12.2 (Pin_2)
- net row4_l: now also J9.1 (Pin_1), RZ1.5 (GP4); no longer J10.1 (Pin_1)
- net row4_r: now also J11.1 (Pin_1), RZ2.5 (GP4); no longer J12.1 (Pin_1)
- net row5_l: now also RZ1.15 (GP14)
- net row5_r: now also RZ2.15 (GP14)
- net scl_l: now also RZ1.3 (GP2)
- net scl_r: now also J2.R1, RZ2.3 (GP2)
- net sda_l: now also J1.R1, RZ1.4 (GP3)
- net sda_r: now also RZ2.4 (GP3)
- new net rst_l: RZ1.2 (GP1), SW1.1
- new net rst_r: RZ2.2 (GP1), SW2.1
- no-connect marks 10 -> 12
Other:
- note added: "Reset button"
- note removed: "For Oled screen, cirque trackpad"
- note removed: "Handedness selection works by pulling a dedicated pin high or low this is checked upon boot and the correct side is set at runtime. The default is high for the left side and low for the right side, but this can be overwritten in firmware."
- note removed: "Power Switch Left"
- note removed: "Power Switch Right"
- note removed: "Pull-ups Left"
- note removed: "Pull-ups Right"
- note removed: "Reset button Left"
- note removed: "Reset button Right"
